File: eagle/atmel_midi_cv_basic.sch (EAGLE design)
At the start: 40 parts, among them IC1 TL074P, U1 ATMEGA328P_PDIP

Commit message: velocity gate led
Parts:
- removed LED1: (no value), SparkFun-LED:LED3MM
- added C4, C6: 100n, rcl:C-US050-024X044
- added IC2: TL074P, linear:TL074P
- added MIDI_CH: 100k, pot:TRIM_US-B64W
- added Q2: 2N3904, transistor-npn:2N3904
- added R4: 1k8, rcl:R-US_0207/10
- added VEL_LED: (no value), SparkFun-LED:LED3MM
- R25: value 4.7k -> 220
Connections:
- removed net N$33: R9.2, U1.PD3(INT1)
- new net N$19: MIDI_CH.S, U1.PC0(ADC0)
- new net N$20: Q2.E, VEL_LED.A
- new net N$21: IC1D.-IN, IC1D.OUT, Q2.C
- new net N$22: R4.2, R9.2, U1.PD3(INT1)
- new net N$23: Q2.B, R4.1
- net +12V: now also C4.1, IC2P.V+
- net +5V: now also MIDI_CH.A, PWR1.+5V
- net -12V: now also C6.2, IC2P.V-
- net GND: now also C4.2, C6.1, MIDI_CH.E
- net N$16: no longer LED1.A
- net N$17: now also IC1D.+IN
- net N$47: now also VEL_LED.C; no longer LED1.C
Other:
- moved on the sheet: C5, C7, C8, C9, PWR1, R17, R25, U$2, U$3

Commit message: board near complete
Parts:
- removed IC2: TL074P, linear:TL074P
- added R10: 1k, rcl:R-US_0207/10
- Q1: device crystal:CRYSTALHC33U-V -> crystal:CRYSTALHC49S
Connections:
- new net N$27: IC1B.OUT, R10.1, R7.2
- net +12V: now also IC1P.V+; no longer IC2P.V+
- net -12V: now also IC1P.V-; no longer IC2P.V-
- net GND: now also PITCH.RING, R6.E, VEL.RING; no longer R6.A
- net N$9: now also R10.2; no longer IC1B.OUT, R7.2
Other:
- moved on the sheet: C4, C5, C6, C7, C8, C9, GATE, IC1A, IC1D, PITCH, PWR1, Q2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

Commit message: almost
Connections:
- net +5V: now also U1.AREF
- net GND: now also U1.PC1(ADC1)
- net N$25: now also U$4.SDI; no longer U$4.SCK
- net N$26: now also U$4.SCK; no longer U$4.SDI
Changed lines of the file:
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@@
 <pinref part="P+1" gate="1" pin="+5V"/>
 <wire x1="-20.32" y1="96.52" x2="-20.32" y2="83.82" width="0.1524" layer="91"/>
+<pinref part="U1" gate="G$1" pin="AREF"/>
+<wire x1="-5.08" y1="58.42" x2="-7.62" y2="58.42" width="0.1524" layer="91"/>
+<wire x1="-7.62" y1="58.42" x2="-7.62" y2="66.04" width="0.1524" layer="91"/>
 </segment>
 <segment>
@@
 <pinref part="GND7" gate="1" pin="GND"/>
 <wire x1="55.88" y1="63.5" x2="55.88" y2="66.04" width="0.1524" layer="91"/>
+<pinref part="U1" gate="G$1" pin="PC1(ADC1)"/>
+<wire x1="43.18" y1="71.12" x2="45.72" y2="71.12" width="0.1524" layer="91"/>
+<wire x1="45.72" y1="71.12" x2="45.72" y2="63.5" width="0.1524" layer="91"/>
+<wire x1="45.72" y1="63.5" x2="55.88" y2="63.5" width="0.1524" layer="91"/>
+<junction x="55.88" y="63.5"/>
 </segment>
 <segment>
@@
 <pinref part="U1" gate="G$1" pin="PB2(SS/OC1B)"/>
 <wire x1="43.18" y1="22.86" x2="63.5" y2="22.86" width="0.1524" layer="91"/>
-<wire x1="63.5" y1="22.86" x2="63.5" y2="121.92" width="0.1524" layer="91"/>
-<pinref part="U$4" gate="A" pin="SCK"/>
-<wire x1="63.5" y1="121.92" x2="83.82" y2="121.92" width="0.1524" layer="91"/>
+<wire x1="63.5" y1="22.86" x2="63.5" y2="119.38" width="0.1524" layer="91"/>
+<pinref part="U$4" gate="A" pin="SDI"/>
+<wire x1="63.5" y1="119.38" x2="83.82" y2="119.38" width="0.1524" layer="91"/>
 </segment>
 </net>
@@
 <pinref part="U1" gate="G$1" pin="PB3(MOSI/OC2)"/>
 <wire x1="43.18" y1="20.32" x2="66.04" y2="20.32" width="0.1524" layer="91"/>
-<wire x1="66.04" y1="20.32" x2="66.04" y2="119.38" width="0.1524" layer="91"/>
-<pinref part="U$4" gate="A" pin="SDI"/>
-<wire x1="66.04" y1="119.38" x2="83.82" y2="119.38" width="0.1524" layer="91"/>
+<wire x1="66.04" y1="20.32" x2="66.04" y2="121.92" width="0.1524" layer="91"/>
 <wire x1="66.04" y1="20.32" x2="78.74" y2="20.32" width="0.1524" layer="91"/>
 <wire x1="78.74" y1="20.32" x2="78.74" y2="27.94" width="0.1524" layer="91"/>
@@
 <pinref part="JP1" gate="G$1" pin="4"/>
 <wire x1="101.6" y1="15.24" x2="93.98" y2="15.24" width="0.1524" layer="91"/>
-</segment>
-</net>
+<pinref part="U$4" gate="A" pin="SCK"/>
+<wire x1="66.04" y1="121.92" x2="83.82" y2="121.92" width="0.1524" layer="91"/>
+</segment>
+</net>
