File: eagle/atmel_midi_cv_2layer.brd (EAGLE design)
At the start: 98.7 x 49.5 mm, 52 parts, among them IC2 TL072P, Q1 16M, U1 ATMEGA328P_PDIP, U2 TLV2372IP

Commit message: layout tweaks
Parts:
- moved R15 9.67 mm to (53.3, 17.8)
- moved R4 8.13 mm to (38.1, 14.0), turned to 90 degrees
Routing:
- net N$39: track 150.7 -> 61.2 mm, vias 0 -> 1
- net N$35: track 57.1 -> 39.0 mm
- net N$1: track 38.1 -> 53.8 mm
- net N$19: track 14.0 -> 3.52 mm
- net +12V: track 49.8 -> 59.0 mm, vias 1 -> 0
- net +5V: track 141.1 -> 146.0 mm
- net N$22: track 33.6 -> 28.9 mm, vias 1 -> 0
- net N$30: track 57.5 -> 54.6 mm
- net N$33: track 24.2 -> 21.7 mm
- net N$24: track 5.07 -> 7.33 mm
- net N$37: track 23.0 -> 21.0 mm
- net -12V: track 27.1 -> 25.5 mm
- net N$28: track 79.4 -> 81.0 mm
- net N$7: track 13.8 -> 15.2 mm
- net N$4: track 15.8 -> 14.9 mm
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