File: eagle/atmel_midi_cv_2layer.sch (EAGLE design)
At the start: 45 parts, among them IC1 TL072P, IC2 TL072P, U1 ATMEGA328P_PDIP

Commit message: rail2rail pitch amp, tone output, improved decoupling, board mount midi jack, more isolation
Parts:
- removed AMT: 100k, pot:3RP/1610N
- removed IC1: TL072P, linear:TL072P
- removed JCK1: AUDIO-JACKITEAD, erthenvar:AUDIO-JACKITEAD
- removed MIDI_CH: 100k, pot:TRIM_US-B64W
- removed MIDI_IN: M02LOCK_LONGPADS, SparkFun-Connectors:M02LOCK_LONGPADS
- removed R11: 1k5, rcl:R-US_0207/7
- removed R5: 3k3, rcl:R-US_0207/7
- removed R7: 5k, rcl:R-US_0207/7
- removed R8: 1k, rcl:R-US_0207/7
- removed RST1, RST2: reset, wirepad:2,54/0,9
- removed SCALE_TRIM: 10k, pot:TRIM_US-B64W
- removed TONE_OUT: AUDIO-JACK, erthenvar:AUDIO-JACK
- added C10: 10u, rcl:CPOL-USB45181A
- added C11, C12, C9: 100n, rcl:C-US050-024X044
- added IN: MIDIJACK, adafruit:MIDIJACK
- added PITCH, TONE: AUDIO-JACKITEAD, erthenvar:AUDIO-JACKITEAD
- added R14: 2k4, rcl:R-US_0207/7
- added R15: 1k, rcl:R-US_0207/7
- added R16: 220, rcl:R-US_0207/7
- added R17: 5k, rcl:R-US_0207/10
- added R18: 1k, rcl:R-US_0207/10
- added R19: 1k2, rcl:R-US_0207/10
- added R6: 20k, rcl:R-US_0207/7
- added RESET: M02LOCK_LONGPADS, SparkFun-Connectors:M02LOCK_LONGPADS
- added SCALE_TRIM1: 10k, pot:TRIM_US-B64W
- added U$1, U$3: FB, adafruit:FB
- added U2: TLV2372IP, Texas Instruments_By_element14_Batch_1:TLV2372IP
- C6: value 100n -> 10u; device rcl:C-US050-024X044 -> rcl:CPOL-USB45181A
- GATE, VEL: value AUDIO-JACK -> AUDIO-JACKITEAD; device erthenvar:AUDIO-JACK -> erthenvar:AUDIO-JACKITEAD
- Q1: value (none) -> 16M
- R12: value 3k9 -> 10k
- R2: value 220 -> 3k3; device rcl:R-US_0207/7 -> rcl:R-US_0207/10
- R9: value 1k5 -> 1k2
Connections:
- removed net N$12: IC1A.-IN, R7.1, SCALE_TRIM.S
- removed net N$13: IC1B.-IN, R11.1, R8.2
- removed net N$14: IC1B.+IN, U$4.VOUTB
- removed net N$2: R5.1, U$4.VOUTA
- removed net N$27: IC1A.OUT, R10.1, R7.2
- removed net N$51: AMT.S, VEL.TIP
- removed net N$6: IC1A.+IN, R5.2
- new net N$32: OK1.VB, R14.1
- new net N$33: ING$1.5
- new net N$34: PWR1.+5V, U$1.1
- new net N$35: IC2A.OUT, R4.1, R6.1
- new net N$36: R2.2, U2.1IN_+
- new net N$37: R17.1, SCALE_TRIM1.S, U2.1IN-
- new net N$38: R18.2, R19.1, U2.2IN-
- new net N$39: R15.1, R19.2, U2.2OUT
- new net N$40: U$4.VOUTB, U2.2IN+
- new net N$41: R10.1, R17.2, U2.1OUT
- net +12V: now also C12.1, U2.VDD; no longer C7.1, IC1P.V+
- net +5V: now also C6.+, C9.1, U$1.2; no longer MIDI_CH.E, PWR1.+5V
- net -12V: now also C10.-, C11.2, U$3.2; no longer PWR1.-12V
- net GND: now also C12.2, C4.2, C6.-, C7.1, C9.2, IC2A.+IN, R18.1, SCALE_TRIM1.E, U2.GND
- net N$17: now also PWR1.-12V, U$3.1; no longer AMT.E, IC1B.OUT, R11.2
- net N$19: now also R15.2, VEL.TIP; no longer MIDI_CH.S, U1.PC0(ADC0)
- net N$20: now also U1.PB1(OC1A); no longer U1.PD6(AIN0)
- net N$21: now also U1.PD7(AIN1); no longer U1.PB5(SCK)
- net N$23: now also R2.1, U$4.VOUTA; no longer IC2A.-IN, IC2A.OUT, R4.1
- net N$24: now also TONE.TIP; no longer TONE_OUT.TIP
- net N$28: now also IC2A.-IN, R6.2; no longer C6.1, IC2A.+IN
- net N$29: now also C10.+, C11.1, PITCH.RING, R14.2, RESET.2, TONE.RING; no longer AMT.A, C4.2, C6.2, IC1P.V-, JCK1.RING, MIDI_CH.A, R8.1, RST2.P, SCALE_TRIM.E, TONE_OUT.RING
- net N$3: no longer MIDI_IN.1
- net N$43: now also RESET.1; no longer RST1.P
- net N$7: now also R16.2; no longer R2.2
- net N$8: now also ING$1.4, R16.1; no longer MIDI_IN.2, R2.1
- net N$9: now also PITCH.TIP; no longer JCK1.TIP
Other:
- moved on the sheet: C4, C5, C7, C8, IC2A, R10, R12, R2, R25, R4, U$2, VEL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

Commit message: merged many 9 to GND
Parts:
- added C13: 100n, rcl:C-US050-024X044
- C3: value .1uF -> 100n
- R17, R19, R2: device rcl:R-US_0207/10 -> rcl:R-US_0207/5V
- R18: device rcl:R-US_0207/10 -> rcl:R-US_0207/7
- R24: device rcl:R-US_0207/7 -> rcl:R-US_0207/5V
- R6, R9: device rcl:R-US_0207/7 -> rcl:R-US_0207/2V
Connections:
- removed net N$29: C1.1, C10.+, C11.1, C2.1, C3.2, C5.-, C8.2, GATE.RING, OK1.GND, PITCH.RING, PWR1.GND, R13.2, R14.2, RESET.2, TONE.RING, U$4.AVSS, U$4.~LDAC, U1.GND@1, U1.GND@2, VEL.RING
- removed net N$3: D1.A, OK1.C
- net +5V: now also C13.1
- net GND: now also C1.1, C10.+, C11.1, C13.2, C2.1, C3.2, C5.-, C8.2, GATE.RING, OK1.GND, PITCH.RING, PWR1.GND, R13.2, R14.2, RESET.2, TONE.RING, U$4.AVSS, U$4.~LDAC, U1.GND@1, U1.GND@2, VEL.RING
- net N$33: now also D1.A, OK1.C

Commit message: started software update
Parts:
- renumbered CV_BUS_ENABLE to BUS_CV, GATE_BUS_ENABLE to BUS_GATE
Changed lines of the file:
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@@
 <grid distance="0.1" unitdist="inch" unit="inch" style="lines" multiple="1" display="no" altdistance="0.01" altunitdist="inch" altunit="inch"/>
 <layers>
-<layer number="1" name="Top" color="4" fill="1" visible="yes" active="no"/>
-<layer number="16" name="Bottom" color="1" fill="1" visible="yes" active="no"/>
-<layer number="17" name="Pads" color="2" fill="1" visible="yes" active="no"/>
-<layer number="18" name="Vias" color="2" fill="1" visible="yes" active="no"/>
-<layer number="19" name="Unrouted" color="6" fill="1" visible="yes" active="no"/>
-<layer number="20" name="Dimension" color="15" fill="1" visible="yes" active="no"/>
-<layer number="21" name="tPlace" color="7" fill="1" visible="yes" active="no"/>
-<layer number="22" name="bPlace" color="7" fill="1" visible="yes" active="no"/>
-<layer number="23" name="tOrigins" color="15" fill="1" visible="yes" active="no"/>
-<layer number="24" name="bOrigins" color="15" fill="1" visible="yes" active="no"/>
-<layer number="25" name="tNames" color="7" fill="1" visible="yes" active="no"/>
-<layer number="26" name="bNames" color="7" fill="1" visible="yes" active="no"/>
-<layer number="27" name="tValues" color="7" fill="1" visible="yes" active="no"/>
-<layer number="28" name="bValues" color="7" fill="1" visible="yes" active="no"/>
+<layer number="1" name="Top" color="4" fill="1" visible="no" active="no"/>
+<layer number="16" name="Bottom" color="1" fill="1" visible="no" active="no"/>
+<layer number="17" name="Pads" color="2" fill="1" visible="no" active="no"/>
+<layer number="18" name="Vias" color="2" fill="1" visible="no" active="no"/>
+<layer number="19" name="Unrouted" color="6" fill="1" visible="no" active="no"/>
+<layer number="20" name="Dimension" color="15" fill="1" visible="no" active="no"/>
+<layer number="21" name="tPlace" color="7" fill="1" visible="no" active="no"/>
+<layer number="22" name="bPlace" color="7" fill="1" visible="no" active="no"/>
+<layer number="23" name="tOrigins" color="15" fill="1" visible="no" active="no"/>
+<layer number="24" name="bOrigins" color="15" fill="1" visible="no" active="no"/>
+<layer number="25" name="tNames" color="7" fill="1" visible="no" active="no"/>
+<layer number="26" name="bNames" color="7" fill="1" visible="no" active="no"/>
+<layer number="27" name="tValues" color="7" fill="1" visible="no" active="no"/>
+<layer number="28" name="bValues" color="7" fill="1" visible="no" active="no"/>
 <layer number="29" name="tStop" color="7" fill="3" visible="no" active="no"/>
 <layer number="30" name="bStop" color="7" fill="6" visible="no" active="no"/>
@@
 <layer number="35" name="tGlue" color="7" fill="4" visible="no" active="no"/>
 <layer number="36" name="bGlue" color="7" fill="5" visible="no" active="no"/>
-<layer number="37" name="tTest" color="7" fill="1" visible="yes" active="no"/>
-<layer number="38" name="bTest" color="7" fill="1" visible="yes" active="no"/>
+<layer number="37" name="tTest" color="7" fill="1" visible="no" active="no"/>
+<layer number="38" name="bTest" color="7" fill="1" visible="no" active="no"/>
 <layer number="39" name="tKeepout" color="4" fill="11" visible="no" active="no"/>
 <layer number="40" name="bKeepout" color="1" fill="11" visible="no" active="no"/>
@@
 <layer number="44" name="Drills" color="7" fill="1" visible="no" active="no"/>
 <layer number="45" name="Holes" color="7" fill="1" visible="no" active="no"/>
-<layer number="46" name="Milling" color="3" fill="1" visible="yes" active="no"/>
-<layer number="47" name="Measures" color="7" fill="1" visible="yes" active="no"/>
-<layer number="48" name="Document" color="7" fill="1" visible="yes" active="no"/>
-<layer number="49" name="Reference" color="7" fill="1" visible="yes" active="no"/>
-<layer number="50" name="dxf" color="7" fill="1" visible="yes" active="no"/>
-<layer number="51" name="tDocu" color="7" fill="1" visible="yes" active="no"/>
-<layer number="52" name="bDocu" color="7" fill="1" visible="yes" active="no"/>
-<layer number="53" name="tGND_GNDA" color="7" fill="9" visible="yes" active="no"/>
-<layer number="54" name="bGND_GNDA" color="1" fill="9" visible="yes" active="no"/>
-<layer number="56" name="wert" color="7" fill="1" visible="yes" active="no"/>
-<layer number="57" name="tCAD" color="7" fill="1" visible="yes" active="no"/>
-<layer number="59" name="tCarbon" color="7" fill="1" visible="yes" active="no"/>
-<layer number="60" name="bCarbon" color="7" fill="1" visible="yes" active="no"/>
+<layer number="46" name="Milling" color="3" fill="1" visible="no" active="no"/>
+<layer number="47" name="Measures" color="7" fill="1" visible="no" active="no"/>
+<layer number="48" name="Document" color="7" fill="1" visible="no" active="no"/>
+<layer number="49" name="Reference" color="7" fill="1" visible="no" active="no"/>
+<layer number="50" name="dxf" color="7" fill="1" visible="no" active="no"/>
+<layer number="51" name="tDocu" color="7" fill="1" visible="no" active="no"/>
+<layer number="52" name="bDocu" color="7" fill="1" visible="no" active="no"/>
+<layer number="53" name="tGND_GNDA" color="7" fill="9" visible="no" active="no"/>
+<layer number="54" name="bGND_GNDA" color="1" fill="9" visible="no" active="no"/>
+<layer number="56" name="wert" color="7" fill="1" visible="no" active="no"/>
+<layer number="57" name="tCAD" color="7" fill="1" visible="no" active="no"/>
+<layer number="59" name="tCarbon" color="7" fill="1" visible="no" active="no"/>
+<layer number="60" name="bCarbon" color="7" fill="1" visible="no" active="no"/>
 <layer number="90" name="Modules" color="5" fill="1" visible="yes" active="yes"/>
 <layer number="91" name="Nets" color="2" fill="1" visible="yes" active="yes"/>
@@
 <part name="P+8" library="supply1" deviceset="+12V" device=""/>
 <part name="C7" library="rcl" deviceset="C-US" device="050-024X044" value="100n"/>
-<part name="GATE_BUS_ENABLE" library="SparkFun-Connectors" deviceset="M02" device="LOCK_LONGPADS"/>
-<part name="CV_BUS_ENABLE" library="SparkFun-Connectors" deviceset="M02" device="LOCK_LONGPADS"/>
+<part name="BUS_GATE" library="SparkFun-Connectors" deviceset="M02" device="LOCK_LONGPADS"/>
+<part name="BUS_CV" library="SparkFun-Connectors" deviceset="M02" device="LOCK_LONGPADS"/>
 <part name="GND13" library="supply1" deviceset="GND" device=""/>
 <part name="P-1" library="supply1" deviceset="-12V" device=""/>
@@
 <instance part="P+8" gate="1" x="91.44" y="40.64"/>
 <instance part="C7" gate="G$1" x="96.52" y="17.78"/>
-<instance part="GATE_BUS_ENABLE" gate="G$1" x="83.82" y="-10.16" rot="R270"/>
-<instance part="CV_BUS_ENABLE" gate="G$1" x="170.18" y="15.24"/>
+<instance part="BUS_GATE" gate="G$1" x="83.82" y="-10.16" rot="R270"/>
+<instance part="BUS_CV" gate="G$1" x="170.18" y="15.24"/>
 <instance part="GND13" gate="1" x="73.66" y="-5.08"/>
 <instance part="P-1" gate="1" x="154.94" y="-10.16"/>
@@
 <wire x1="185.42" y1="88.9" x2="185.42" y2="106.68" width="0.1524" layer="91"/>
 <junction x="185.42" y="106.68"/>
-<pinref part="CV_BUS_ENABLE" gate="G$1" pin="2"/>
+<pinref part="BUS_CV" gate="G$1" pin="2"/>
 <wire x1="177.8" y1="17.78" x2="205.74" y2="17.78" width="0.1524" layer="91"/>
 <pinref part="PITCH" gate="G$1" pin="TIP"/>
@@
 <wire x1="45.72" y1="-20.32" x2="83.82" y2="-20.32" width="0.1524" layer="91"/>
 <pinref part="GATE" gate="G$1" pin="TIP"/>
-<pinref part="GATE_BUS_ENABLE" gate="G$1" pin="1"/>
+<pinref part="BUS_GATE" gate="G$1" pin="1"/>
 <wire x1="83.82" y1="-17.78" x2="83.82" y2="-20.32" width="0.1524" layer="91"/>
 </segment>
@@
 <wire x1="116.84" y1="-20.32" x2="116.84" y2="-15.24" width="0.1524" layer="91"/>
 <wire x1="86.36" y1="-20.32" x2="116.84" y2="-20.32" width="0.1524" layer="91"/>
-<pinref part="GATE_BUS_ENABLE" gate="G$1" pin="2"/>
+<pinref part="BUS_GATE" gate="G$1" pin="2"/>
 <wire x1="86.36" y1="-17.78" x2="86.36" y2="-20.32" width="0.1524" layer="91"/>
 </segment>
@@
 <net name="N$15" class="0">
 <segment>
-<pinref part="CV_BUS_ENABLE" gate="G$1" pin="1"/>
+<pinref part="BUS_CV" gate="G$1" pin="1"/>
 <wire x1="177.8" y1="15.24" x2="180.34" y2="15.24" width="0.1524" layer="91"/>
 <wire x1="180.34" y1="-33.02" x2="180.34" y2="15.24" width="0.1524" layer="91"/>

Commit message: added url and release to silkscreen
Parts:
- R17, R19, R2, R24: device rcl:R-US_0207/5V -> rcl:R-US_0207/7
- R6, R9: device rcl:R-US_0207/2V -> rcl:R-US_0207/7
- VEL_LED: device SparkFun-LED:LED5MM -> SparkFun-LED:LED3MM
- renumbered SCALE_TRIM1 to SCALE
Changed lines of the file:
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@@
 <part name="GND10" library="supply1" deviceset="GND" device=""/>
 <part name="GND9" library="supply1" deviceset="GND" device=""/>
-<part name="R24" library="rcl" deviceset="R-US_" device="0207/5V" value="1M"/>
+<part name="R24" library="rcl" deviceset="R-US_" device="0207/7" value="1M"/>
 <part name="R25" library="rcl" deviceset="R-US_" device="0207/7" value="470"/>
-<part name="VEL_LED" library="SparkFun-LED" deviceset="LED" device="5MM"/>
-<part name="R9" library="rcl" deviceset="R-US_" device="0207/2V" value="1k2"/>
+<part name="VEL_LED" library="SparkFun-LED" deviceset="LED" device="3MM"/>
+<part name="R9" library="rcl" deviceset="R-US_" device="0207/7" value="1k2"/>
 <part name="R26" library="rcl" deviceset="R-US_" device="0207/7" value="1k"/>
 <part name="GND14" library="supply1" deviceset="GND" device=""/>
@@
 <part name="P-2" library="supply1" deviceset="-12V" device=""/>
 <part name="PITCH" library="erthenvar" deviceset="AUDIO-JACK" device="ITEAD"/>
-<part name="R6" library="rcl" deviceset="R-US_" device="0207/2V" value="20k"/>
+<part name="R6" library="rcl" deviceset="R-US_" device="0207/7" value="20k"/>
 <part name="R14" library="rcl" deviceset="R-US_" device="0207/7" value="2k4"/>
 <part name="C6" library="rcl" deviceset="CPOL-US" device="B45181A" value="10u"/>
@@
 <part name="IN" library="adafruit" deviceset="MIDIJACK" device=""/>
 <part name="RESET" library="SparkFun-Connectors" deviceset="M02" device="LOCK_LONGPADS"/>
-<part name="R2" library="rcl" deviceset="R-US_" device="0207/5V" value="3k3"/>
-<part name="SCALE_TRIM1" library="pot" deviceset="TRIM_US-" device="B64W" value="10k"/>
-<part name="R17" library="rcl" deviceset="R-US_" device="0207/5V" value="5k"/>
+<part name="R2" library="rcl" deviceset="R-US_" device="0207/7" value="3k3"/>
+<part name="SCALE" library="pot" deviceset="TRIM_US-" device="B64W" value="10k"/>
+<part name="R17" library="rcl" deviceset="R-US_" device="0207/7" value="5k"/>
 <part name="R18" library="rcl" deviceset="R-US_" device="0207/7" value="1k"/>
-<part name="R19" library="rcl" deviceset="R-US_" device="0207/5V" value="1k2"/>
+<part name="R19" library="rcl" deviceset="R-US_" device="0207/7" value="1k2"/>
 <part name="P+3" library="supply1" deviceset="+12V" device=""/>
 <part name="GND7" library="supply1" deviceset="GND" device=""/>
@@
 </instance>
 <instance part="R2" gate="G$1" x="119.38" y="116.84"/>
-<instance part="SCALE_TRIM1" gate="G$1" x="104.14" y="81.28" rot="MR180"/>
+<instance part="SCALE" gate="G$1" x="104.14" y="81.28" rot="MR180"/>
 <instance part="R17" gate="G$1" x="147.32" y="129.54"/>
 <instance part="R18" gate="G$1" x="116.84" y="76.2"/>
@@
 </segment>
 <segment>
-<pinref part="SCALE_TRIM1" gate="G$1" pin="E"/>
+<pinref part="SCALE" gate="G$1" pin="E"/>
 <wire x1="104.14" y1="73.66" x2="104.14" y2="66.04" width="0.1524" layer="91"/>
 <pinref part="GND18" gate="1" pin="GND"/>
@@
 <wire x1="142.24" y1="129.54" x2="119.38" y2="129.54" width="0.1524" layer="91"/>
 <wire x1="119.38" y1="129.54" x2="119.38" y2="99.06" width="0.1524" layer="91"/>
-<pinref part="SCALE_TRIM1" gate="G$1" pin="S"/>
+<pinref part="SCALE" gate="G$1" pin="S"/>
 <wire x1="109.22" y1="81.28" x2="119.38" y2="81.28" width="0.1524" layer="91"/>
 <wire x1="119.38" y1="81.28" x2="119.38" y2="99.06" width="0.1524" layer="91"/>

Commit message: ICSP added and rerouted
Parts:
- added SV1: (no value), con-lstb:MA03-2
Connections:
- new net N$2: SV1.3, U1.PB5(SCK)
- net +5V: now also SV1.2
- net GND: now also SV1.6
- net N$25: now also SV1.4
- net N$43: now also SV1.5
- net N$45: now also SV1.1
Changed lines of the file:
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@@
 <?xml version="1.0" encoding="utf-8"?>
 <!DOCTYPE eagle SYSTEM "eagle.dtd">
-<eagle version="7.6.0">
+<eagle version="8.3.2">
 <drawing>
 <settings>
 <setting alwaysvectorfont="no"/>
+<setting keepoldvectorfont="yes"/>
 <setting verticaltext="up"/>
 </settings>
@@
 <part name="C13" library="rcl" deviceset="C-US" device="050-024X044" value="100n"/>
 <part name="GND19" library="supply1" deviceset="GND" device=""/>
+<part name="SV1" library="con-lstb" library_urn="urn:adsk.eagle:library:162" deviceset="MA03-2" device="" package3d_urn="urn:adsk.eagle:package:8334/1"/>
+<part name="P+4" library="supply1" deviceset="+5V" device=""/>
+<part name="GND20" library="supply1" deviceset="GND" device=""/>
 </parts>
 <sheets>
@@
 <instance part="C13" gate="G$1" x="58.42" y="124.46"/>
 <instance part="GND19" gate="1" x="58.42" y="114.3"/>
+<instance part="SV1" gate="1" x="81.28" y="68.58" rot="R180"/>
+<instance part="P+4" gate="1" x="88.9" y="78.74"/>
+<instance part="GND20" gate="1" x="88.9" y="55.88"/>
 </instances>
 <busses>
@@
 <junction x="149.86" y="-15.24"/>
 </segment>
+<segment>
+<pinref part="SV1" gate="1" pin="2"/>
+<pinref part="P+4" gate="1" pin="+5V"/>
+<wire x1="88.9" y1="76.2" x2="88.9" y2="71.12" width="0.1524" layer="91"/>
+</segment>
 </net>
 <net name="+12V" class="0">
@@
 <net name="N$25" class="0">
 <segment>
-<wire x1="66.04" y1="20.32" x2="66.04" y2="109.22" width="0.1524" layer="91"/>
+<wire x1="66.04" y1="20.32" x2="66.04" y2="81.28" width="0.1524" layer="91"/>
 <pinref part="U$4" gate="A" pin="SCK"/>
+<wire x1="66.04" y1="81.28" x2="66.04" y2="109.22" width="0.1524" layer="91"/>
 <wire x1="66.04" y1="109.22" x2="76.2" y2="109.22" width="0.1524" layer="91"/>
 <pinref part="U1" gate="G$1" pin="PB3(MOSI/OC2)"/>
 <wire x1="66.04" y1="20.32" x2="43.18" y2="20.32" width="0.1524" layer="91"/>
+<pinref part="SV1" gate="1" pin="4"/>
+<wire x1="88.9" y1="68.58" x2="93.98" y2="68.58" width="0.1524" layer="91"/>
+<wire x1="93.98" y1="68.58" x2="93.98" y2="81.28" width="0.1524" layer="91"/>
+<wire x1="93.98" y1="81.28" x2="66.04" y2="81.28" width="0.1524" layer="91"/>
+<junction x="66.04" y="81.28"/>
 </segment>
 </net>
@@
 <wire x1="-7.62" y1="83.82" x2="-10.16" y2="83.82" width="0.1524" layer="91"/>
 <wire x1="-5.08" y1="73.66" x2="-7.62" y2="73.66" width="0.1524" layer="91"/>
-<wire x1="-7.62" y1="73.66" x2="-7.62" y2="83.82" width="0.1524" layer="91"/>
+<wire x1="-7.62" y1="73.66" x2="-7.62" y2="78.74" width="0.1524" layer="91"/>
 <junction x="-7.62" y="83.82"/>
 <pinref part="RESET" gate="G$1" pin="1"/>
+<wire x1="-7.62" y1="83.82" x2="-7.62" y2="78.74" width="0.1524" layer="91"/>
+<wire x1="-7.62" y1="78.74" x2="71.12" y2="78.74" width="0.1524" layer="91"/>
+<wire x1="71.12" y1="78.74" x2="71.12" y2="66.04" width="0.1524" layer="91"/>
+<pinref part="SV1" gate="1" pin="5"/>
+<wire x1="71.12" y1="66.04" x2="73.66" y2="66.04" width="0.1524" layer="91"/>
+<junction x="-7.62" y="78.74"/>
 </segment>
 </net>
@@
 <wire x1="43.18" y1="17.78" x2="68.58" y2="17.78" width="0.1524" layer="91"/>
 <pinref part="U$4" gate="A" pin="~CS"/>
-<wire x1="68.58" y1="17.78" x2="68.58" y2="111.76" width="0.1524" layer="91"/>
+<wire x1="68.58" y1="17.78" x2="68.58" y2="71.12" width="0.1524" layer="91"/>
+<wire x1="68.58" y1="71.12" x2="68.58" y2="111.76" width="0.1524" layer="91"/>
 <wire x1="68.58" y1="111.76" x2="76.2" y2="111.76" width="0.1524" layer="91"/>
+<pinref part="SV1" gate="1" pin="1"/>
+<wire x1="73.66" y1="71.12" x2="68.58" y2="71.12" width="0.1524" layer="91"/>
+<junction x="68.58" y="71.12"/>
 </segment>
 </net>
@@
 <pinref part="R13" gate="G$1" pin="2"/>
 </segment>
+<segment>
+<pinref part="SV1" gate="1" pin="6"/>
+<pinref part="GND20" gate="1" pin="GND"/>
+<wire x1="88.9" y1="58.42" x2="88.9" y2="66.04" width="0.1524" layer="91"/>
+</segment>
 </net>
 <net name="-12V" class="0">
@@
 </segment>
 </net>
+<net name="N$2" class="0">
+<segment>
+<pinref part="U1" gate="G$1" pin="PB5(SCK)"/>
+<wire x1="43.18" y1="15.24" x2="60.96" y2="15.24" width="0.1524" layer="91"/>
+<wire x1="60.96" y1="15.24" x2="60.96" y2="68.58" width="0.1524" layer="91"/>
+<pinref part="SV1" gate="1" pin="3"/>
+<wire x1="60.96" y1="68.58" x2="73.66" y2="68.58" width="0.1524" layer="91"/>
+</segment>
+</net>
 </nets>
 </sheet>
@@
 </schematic>
 </drawing>
+<compatibility>
+<note version="8.2" severity="warning">
+Since Version 8.2, EAGLE supports online libraries. The ids
+of those online libraries will not be understood (or retained)
+with this version.
+</note>
+<note version="8.3" severity="warning">
+Since Version 8.3, EAGLE supports URNs for individual library
+assets (packages, symbols, and devices). The URNs of those assets
+will not be understood (or retained) with this version.
+</note>
+<note version="8.3" severity="warning">
+Since Version 8.3, EAGLE supports the association of 3D packages
+with devices in libraries, schematics, and board files. Those 3D
+packages will not be understood (or retained) with this version.
+</note>
+</compatibility>
 </eagle>

Commit message: updated power with shroud
Changed lines of the file:
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@@
 <?xml version="1.0" encoding="utf-8"?>
 <!DOCTYPE eagle SYSTEM "eagle.dtd">
-<eagle version="8.3.2">
+<eagle version="7.6.0">
 <drawing>
 <settings>
 <setting alwaysvectorfont="no"/>
-<setting keepoldvectorfont="yes"/>
 <setting verticaltext="up"/>
 </settings>
@@
 <part name="C13" library="rcl" deviceset="C-US" device="050-024X044" value="100n"/>
 <part name="GND19" library="supply1" deviceset="GND" device=""/>
-<part name="SV1" library="con-lstb" library_urn="urn:adsk.eagle:library:162" deviceset="MA03-2" device="" package3d_urn="urn:adsk.eagle:package:8334/1"/>
+<part name="SV1" library="con-lstb" deviceset="MA03-2" device=""/>
 <part name="P+4" library="supply1" deviceset="+5V" device=""/>
 <part name="GND20" library="supply1" deviceset="GND" device=""/>
@@
 </schematic>
 </drawing>
-<compatibility>
-<note version="8.2" severity="warning">
-Since Version 8.2, EAGLE supports online libraries. The ids
-of those online libraries will not be understood (or retained)
-with this version.
-</note>
-<note version="8.3" severity="warning">
-Since Version 8.3, EAGLE supports URNs for individual library
-assets (packages, symbols, and devices). The URNs of those assets
-will not be understood (or retained) with this version.
-</note>
-<note version="8.3" severity="warning">
-Since Version 8.3, EAGLE supports the association of 3D packages
-with devices in libraries, schematics, and board files. Those 3D
-packages will not be understood (or retained) with this version.
-</note>
-</compatibility>
 </eagle>
